Commit message: [nextagea_description] Set default behaviour to be fixed base

File: nextagea_description/urdf/nxao_gz.xacro (robot description, xacro)
@@ -2,5 +2,5 @@
 <robot name="NextageAOpen"
        xmlns:xacro="http://www.ros.org/wiki/xacro">
-  <xacro:property name="fixed_base" value="False" />
+  <xacro:property name="fixed_base" value="True" />
   <xacro:include filename="$(find nextagea_description)/urdf/NextageAOpen.urdf" />
   <xacro:include filename="$(find nextagea_description)/urdf/nxao_gz_camera.xacro" />

Commit message: [nextagea_gazebo] Add and configure hand cameras on each arm

File: nextagea_description/urdf/nxao_gz.xacro (robot description, xacro)
@@ -11,10 +11,12 @@
   <xacro:property name="jnt_head_camera_rot_y" value="0.25" />
   <xacro:property name="link_head_camera_rot_z" value="0.05" />
-  <!-- NOTE: The poses of headmount cameras are NOT precisely adjusted to
+  <xacro:property name="jnt_hand_camera_displacement_x" value="0.0525" />
+  <xacro:property name="jnt_hand_camera_displacement_y" value="0.0525" />
+  <xacro:property name="jnt_hand_camera_displacement_z" value="0.0" />
+  <xacro:property name="jnt_hand_camera_rot_y" value="1.5708" />
+  <xacro:property name="link_hand_camera_rot_z" value="0.0" />
+  <!-- NOTE: The poses of headmount and hand cameras are NOT precisely adjusted to
              the 3D model nor the actual hardware config. These configs
-             are meant for a rapid prototyping only. If you need precise
-             configuration, please go ahead modify the following, then
-             (if possible) send a patch to https://github.com/tork-a/rtmros_nextage/pulls
-             so that other developers and users can use (and possible improve).
+             are meant for a rapid prototyping only.
   -->
   <xacro:camera_joint_link_gzplugin
@@ -30,6 +32,16 @@
          link_displacement_x="0.0325" link_displacement_y="0" link_displacement_z="0"
          link_rotation_x="0" link_rotation_y="${M_PI/2}" link_rotation_z="${link_head_camera_rot_z}" />
-  <!-- TODO hand cameras can be added here with the very similar code as
-            headmount cameras. -->
+  <xacro:camera_joint_link_gzplugin
+         camera_name="CAMERA_HAND_L" link_parent="LARM_JOINT5_Link"
+         jnt_displacement_x="${jnt_hand_camera_displacement_x}" jnt_displacement_y="${jnt_hand_camera_displacement_y}" jnt_displacement_z="${jnt_hand_camera_displacement_z}"
+         jnt_rotation_x="0" jnt_rotation_y="${jnt_hand_camera_rot_y}" jnt_rotation_z="0"
+         link_displacement_x="0.0325" link_displacement_y="0" link_displacement_z="0"
+         link_rotation_x="0" link_rotation_y="${M_PI/2}" link_rotation_z="-${link_hand_camera_rot_z}" />
+  <xacro:camera_joint_link_gzplugin
+         camera_name="CAMERA_HAND_R" link_parent="RARM_JOINT5_Link"
+         jnt_displacement_x="${jnt_hand_camera_displacement_x}" jnt_displacement_y="-${jnt_hand_camera_displacement_y}" jnt_displacement_z="${jnt_hand_camera_displacement_z}"
+         jnt_rotation_x="0" jnt_rotation_y="${jnt_hand_camera_rot_y}" jnt_rotation_z="0"
+         link_displacement_x="0.0325" link_displacement_y="0" link_displacement_z="0"
+         link_rotation_x="0" link_rotation_y="${M_PI/2}" link_rotation_z="-${link_hand_camera_rot_z}" />
   <!-- Gazebo-Specific Link Properties -->
   <gazebo reference="CHEST_JOINT0">
