Commit message: [nextagea_description] fixed base in gazebo

File: nextagea_description/urdf/NextageAOpen.urdf (robot description, URDF)
Before this commit: robot NextageAOpen, 16 links, 15 joints
Links:
- added link world
Joints:
- added joint fixed: type fixed, parent world, child WAIST

Commit message: [nextagea_description] Make gazebo fixed joint optional

File: nextagea_description/urdf/NextageAOpen.urdf (robot description, URDF)
Before this commit: robot NextageAOpen, 17 links, 16 joints
Links:
- removed link world
Joints:
- removed joint fixed

File: nextagea_description/urdf/nxao_gz.xacro (robot description, xacro)
@@ -2,4 +2,5 @@
 <robot name="NextageAOpen"
        xmlns:xacro="http://www.ros.org/wiki/xacro">
+  <xacro:property name="fixed_base" value="False" />
   <xacro:include filename="$(find nextagea_description)/urdf/NextageAOpen.urdf" />
   <xacro:include filename="$(find nextagea_description)/urdf/nxao_gz_camera.xacro" />

Commit message: [nextagea_description] Replaced collision meshes with shape primitives

File: nextagea_description/urdf/NextageAOpen.urdf (robot description, URDF)
Before this commit: robot NextageAOpen, 16 links, 15 joints
Links:
- link CHEST_JOINT0_Link: geometry collision box size=0.085 0.5 0.0365; collision box size=0.17 0.29 0.225
- link HEAD_JOINT0_Link: geometry collision cylinder length=0.135 radius=0.035; visual mesh filename=package://nextagea_description/urdf/meshes/HEAD_JOINT0_Link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
- link HEAD_JOINT1_Link: geometry collision box size=0.27 0.22 0.115; visual mesh filename=package://nextagea_description/urdf/meshes/HEAD_JOINT1_Link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
- link LARM_JOINT0_Link: geometry collision box size=0.048 0.1 0.035; collision box size=0.1 0.0815 0.19
- link LARM_JOINT1_Link: geometry collision box size=0.08 0.11 0.28; collision box size=0.122 0.0338 0.062
- link LARM_JOINT2_Link: geometry collision box size=0.119 0.125 0.1; collision cylinder length=0.04 radius=0.047
- link LARM_JOINT3_Link: geometry collision box size=0.093 0.112 0.037; collision cylinder length=0.12 radius=0.035
- link LARM_JOINT4_Link: geometry collision box size=0.04 0.118 0.06; collision cylinder length=0.08 radius=0.037
- link LARM_JOINT5_Link: geometry collision box size=0.057 0.106 0.042; collision cylinder length=0.07 radius=0.037
- link RARM_JOINT0_Link: geometry collision box size=0.048 0.1 0.035; collision box size=0.1 0.0815 0.19
- link RARM_JOINT1_Link: geometry collision box size=0.08 0.11 0.28; collision box size=0.122 0.0338 0.062
- link RARM_JOINT2_Link: geometry collision box size=0.119 0.125 0.1; collision cylinder length=0.04 radius=0.047
- link RARM_JOINT3_Link: geometry collision box size=0.093 0.112 0.037; collision cylinder length=0.12 radius=0.035
- link RARM_JOINT4_Link: geometry collision box size=0.04 0.118 0.06; collision cylinder length=0.08 radius=0.037
- link RARM_JOINT5_Link: geometry collision box size=0.057 0.106 0.042; collision cylinder length=0.07 radius=0.037
- link WAIST: geometry collision box size=0.585 0.585 0.72; collision cylinder length=0.376 radius=0.06

Commit message: [nextagea_description] Add a dummy link "nextage_base" to work around KDL issue - Root link cannot have a mass. - This is not equivalent to fixing it in Gazebo.

File: nextagea_description/urdf/NextageAOpen.urdf (robot description, URDF)
Before this commit: robot NextageAOpen, 16 links, 15 joints
Links:
- added link nextage_base
Joints:
- added joint base_to_waist: type fixed, parent nextage_base, child WAIST

Commit message: [nextagea_description] Add joint velocity and acceleration limits

File: nextagea_description/urdf/NextageAOpen.urdf (robot description, URDF)
Before this commit: robot NextageAOpen, 17 links, 16 joints
Joints:
- joint LARM_JOINT0: limit lower=-1.5707963 upper=1.5707963 effort=150 velocity=1.0 -> lower=-1.5707963 upper=1.5707963 effort=150 velocity=2.0
- joint LARM_JOINT1: limit lower=-2.44346 upper=1.0471975 effort=150 velocity=1.0 -> lower=-2.44346 upper=1.0471975 effort=150 velocity=2.0

Commit message: [nextagea_gazebo] Adjust accel rates

File: nextagea_description/urdf/NextageAOpen.urdf (robot description, URDF)
Before this commit: robot NextageAOpen, 17 links, 16 joints
Joints:
- joint LARM_JOINT0: limit lower=-1.5707963 upper=1.5707963 effort=150 velocity=2.0 -> lower=-1.5707963 upper=1.5707963 effort=150 velocity=1.0
- joint LARM_JOINT1: limit lower=-2.44346 upper=1.0471975 effort=150 velocity=2.0 -> lower=-2.44346 upper=1.0471975 effort=150 velocity=1.0
