Commit message: set world frame to ground plane

File: nextagea_description/urdf/NextageAOpen_gazebo.urdf.xacro (robot description, xacro)
@@ -12,5 +12,5 @@
       <parent link="world"/>
       <child link="base_link"/>
-      <origin xyz="0 0 -0.15" rpy="0 0 0"/>
+      <origin xyz="0 0 0.85" rpy="0 0 0"/>
     </joint>
   </xacro:if>
