Commit message: URDF restructuring (#11)
* [nextagea_description] Split base model and restructured xacros

* [nextagea_gazebo] change to position control, re-tuned gains, fixed up scripts

* PR fixes

File: nextagea_description/urdf/NextageA_robot.xacro (robot description, xacro)
@@ -1,57 +1,5 @@
 <?xml version="1.0"?>
-<robot name="NextageAOpen"
-       xmlns:xi="http://www.w3.org/2001/xinclude"
-       xmlns:gazebo="http://playerstage.sourceforge.net/gazebo/xmlschema/#gz"
-       xmlns:model="http://playerstage.sourceforge.net/gazebo/xmlschema/#model"
-       xmlns:sensor="http://playerstage.sourceforge.net/gazebo/xmlschema/#sensor"
-       xmlns:body="http://playerstage.sourceforge.net/gazebo/xmlschema/#body"
-       xmlns:geom="http://playerstage.sourceforge.net/gazebo/xmlschema/#geom"
-       xmlns:joint="http://playerstage.sourceforge.net/gazebo/xmlschema/#joint"
-       xmlns:interface="http://playerstage.sourceforge.net/gazebo/xmlschema/#interface"
-       xmlns:rendering="http://playerstage.sourceforge.net/gazebo/xmlschema/#rendering"
-       xmlns:renderable="http://playerstage.sourceforge.net/gazebo/xmlschema/#renderable"
-       xmlns:controller="http://playerstage.sourceforge.net/gazebo/xmlschema/#controller"
-       xmlns:physics="http://playerstage.sourceforge.net/gazebo/xmlschema/#physics"
-       xmlns:xacro="http://www.ros.org/wiki/xacro">
-  <xacro:include filename="$(find nextagea_description)/urdf/materials.urdf.xacro" />
-  <xacro:macro name="transmission_nx_joint" params="name">
-    <transmission name="${name}_Trans">
-      <type>transmission_interface/SimpleTransmission</type>
-      <joint name="${name}">
-        <hardwareInterface>hardware_interface/EffortJointInterface</hardwareInterface>/hardwareInterface>
-      </joint>
-      <actuator name="${name}_Motor">
-        <hardwareInterface>hardware_interface/EffortJointInterface</hardwareInterface>/hardwareInterface>
-        <mechanicalReduction>1</mechanicalReduction>
-      </actuator>
-    </transmission>
-  </xacro:macro>
-  <!-- Define contact properties -->
-  <xacro:macro name="gazebo_nx_link" params="name color">
-    <gazebo reference="gazebo_${name}">
-      <material>Gazebo/${color}</material>
-      <mu1 value="1.0" />
-      <mu2 value="1.0" />
-      <kp  value="1000000.0" />
-      <kd  value="100.0" />
-      <maxVel  value="100.0" />
-      <minDepth  value="0.0" />
-    </gazebo>
-  </xacro:macro>
-  <!-- Used for fixing robot to Gazebo 'base_link' -->
-  <xacro:if value="${fixed_base}">
-    <link name="world"/> -->
-    <joint name="fixed" type="fixed">
-      <parent link="world"/>
-      <child link="nextage_base"/>
-      <origin xyz="0 0 -0.15" rpy="0 0 0"/>
-    </joint>
-  </xacro:if>
-  <!-- Work-around for KDL base-link inertia problem; also adheres to ROS standard-->
-  <link name="nextage_base"/>
-  <joint name="base_to_waist" type="fixed">
-    <parent link="nextage_base"/>
-    <child link="WAIST"/>
-  </joint>
+<robot xmlns:xacro="http://ros.org/wiki/xacro">
+  <xacro:include filename="$(find nextagea_description)/urdf/common.xacro" />
   <xacro:gazebo_nx_link name="WAIST" color="Black" />
   <link name="WAIST">
@@ -63,34 +11,4 @@
     </visual>
     <collision>
-      <origin xyz="-0.19 0 -0.435" rpy="0 0 0"/>
-      <geometry>
-        <box size="0.585 0.585 0.72"/>
-      </geometry>
-    </collision>
-    <collision>
-      <origin xyz="0.0675 0.2575 -0.82" rpy="0 0 0"/>
-      <geometry>
-        <sphere radius="0.03"/>
-      </geometry>
-    </collision>
-    <collision>
-      <origin xyz="0.0675 -0.2575 -0.82" rpy="0 0 0"/>
-      <geometry>
-        <sphere radius="0.03"/>
-      </geometry>
-    </collision>
-    <collision>
-      <origin xyz="-0.4475 0.2575 -0.82" rpy="0 0 0"/>
-      <geometry>
-        <sphere radius="0.03"/>
-      </geometry>
-    </collision>
-    <collision>
-      <origin xyz="-0.4475 -0.2575 -0.82" rpy="0 0 0"/>
-      <geometry>
-        <sphere radius="0.03"/>
-      </geometry>
-    </collision>
-    <collision>
       <origin xyz="0.0 0 0.098" rpy="0 0 0"/>
       <geometry>
@@ -99,7 +17,7 @@
     </collision>
     <inertial>
-      <mass value="10000" />
-      <origin xyz="0 0 0" rpy="0 -0 0"/>
-      <inertia ixx="20" ixy="0" ixz="0" iyy="20" iyz="0" izz="20"/>
+      <mass value="5" />
+      <origin xyz="0 0 0.15" rpy="0 0 0"/>
+      <xacro:nxa_box_inertia_def x="0.2" y="0.2" z="0.3" mass="5"/>
     </inertial>
   </link>
@@ -155,7 +73,7 @@
     </collision>
     <inertial>
-      <mass value="3.0" />
-      <origin xyz="0 0 0" rpy="0 -0 0"/>
-      <inertia ixx="0.0639575" ixy="-0.00022833" ixz="0.00011172" iyy="0.0310845" iyz="6.48e-05" izz="0.0501107"/>
+      <mass value="10.0" />
+      <origin xyz="0 0 0.2" rpy="0 -0 0"/>
+      <xacro:nxa_box_inertia_def x="0.25" y="0.25" z="0.3" mass="10"/>
     </inertial>
   </link>
@@ -176,6 +94,6 @@
      <inertial>
       <mass value="0.317929" />
-      <origin xyz="-2.292e-05 0.00547848 -0.00784016" rpy="0 -0 0"/>
-      <inertia ixx="0.00027682" ixy="3e-08" ixz="-3.3e-07" iyy="0.00013009" iyz="-1.092e-05" izz="0.00020954"/>
+      <origin xyz="0 0.00547848 0" rpy="0 -0 0"/>
+      <xacro:nxa_box_inertia_def x="0.1" y="0.1" z="0.1" mass="0.317929"/>
     </inertial>
   </link>
@@ -195,8 +113,7 @@
     </collision>
     <inertial>
-      <mass value="0.0808593" />
-      <!-- <origin xyz="5.02e-06 -0.0166777 0.0163153" rpy="0 -0 0"/> -->
-      <!-- <inertia ixx="8.07e-05" ixy="-3e-08" ixz="-4.30134e-22" iyy="3.025e-05" iyz="-1.277e-05" izz="6.637e-05"/> -->
-      <inertia ixx="1e-3" ixy="0" ixz="0" iyy="1e-3" iyz="0" izz="1e-3"/>
+      <mass value="0.4" />
+      <origin xyz="-0.05 0 0.12" rpy="0 0.26 0"/>
+      <xacro:nxa_box_inertia_def x="0.27" y="0.22" z="0.115" mass="0.4"/>
     </inertial>
   </link>
@@ -229,5 +146,5 @@
     <inertial>
       <mass value="1.32626" />
-      <origin xyz="-0.00226388 -0.00521383 0.0156081" rpy="0 -0 0"/>
+      <origin xyz="0.0 0.05 0.05" rpy="0 -0 0"/>
       <inertia ixx="0.00207537" ixy="0.00011276" ixz="8.927e-05" iyy="0.00240295" iyz="-4.57e-05" izz="0.00141912"/>
     </inertial>
@@ -255,6 +172,6 @@
      <inertial>
       <mass value="1.14898" />
-      <origin xyz="-5.236e-05 0.0583134 -0.107061" rpy="0 -0 0"/>
-    <inertia ixx="0.0154168" ixy="9.95417e-07" ixz="3.38147e-06" iyy="0.0147117" iyz="0.00213719" izz="0.0012658"/>
+      <origin xyz="-0.04 0.1 -0.12" rpy="0 -0 0"/>
+      <inertia ixx="0.0154168" ixy="9.95417e-07" ixz="3.38147e-06" iyy="0.0147117" iyz="0.00213719" izz="0.0012658"/>
     </inertial>
   </link>
@@ -287,5 +204,5 @@
     <inertial>
       <mass value="0.577518" />
-      <origin xyz="-2.254e-05 0.00167107 -0.0715116" rpy="0 -0 0"/>
+      <origin xyz="0.1 0.01167107 -0.04" rpy="0 -0 0"/>
       <inertia ixx="0.00143966" ixy="-3e-07" ixz="1.2e-06" iyy="0.00141763" iyz="-7.596e-05" izz="0.0001972"/>
     </inertial>
@@ -319,5 +236,5 @@
     <inertial>
       <mass value="0.457418" />
-      <origin xyz="-1.788e-05 -0.00395812 -0.20273" rpy="0 -0 0"/>
+      <origin xyz="0.1 -0.00395812 -0.00273" rpy="0 -0 0"/>
       <inertia ixx="0.00069205" ixy="3e-08" ixz="5.2e-07" iyy="0.00068903" iyz="-1.915e-05" izz="0.00013509"/>
     </inertial>
@@ -377,5 +294,5 @@
     <inertial>
       <mass value="1.05156" />
-      <origin xyz="-0.048476 -3.2e-06 -0.0388988" rpy="0 -0 0"/>
+      <origin xyz="0.0 0.0 -0.08" rpy="0 -0 0"/>
       <inertia ixx="0.00194072" ixy="1.1e-07" ixz="-0.00042482" iyy="0.00209392" iyz="1.2e-07" izz="0.00035788"/>
     </inertial>
@@ -409,5 +326,5 @@
     <inertial>
       <mass value="1.32626" />
-      <origin xyz="-0.00226388 0.00521383 0.0156081" rpy="0 -0 0"/>
+      <origin xyz="0.0 -0.05 0.05" rpy="0 -0 0"/>
       <inertia ixx="0.00207537" ixy="-0.00011276" ixz="8.927e-05" iyy="0.00240295" iyz="4.57e-05" izz="0.00141912"/>
     </inertial>
@@ -435,5 +352,5 @@
     <inertial>
       <mass value="1.14898" />
-      <origin xyz="-5.236e-05 -0.0583134 -0.107061" rpy="0 -0 0"/>
+      <origin xyz="-0.04 -0.1 -0.12" rpy="0 -0 0"/>
       <inertia ixx="0.0154168" ixy="-9.95417e-07" ixz="3.38147e-06" iyy="0.0147117" iyz="-0.00213719" izz="0.0012658"/>
     </inertial>
@@ -467,5 +384,5 @@
     <inertial>
       <mass value="0.577518" />
-      <origin xyz="-2.254e-05 -0.00167107 -0.0715116" rpy="0 -0 0"/>
+      <origin xyz="0.1 -0.01167107 -0.04" rpy="0 -0 0"/>
       <inertia ixx="0.00143966" ixy="3e-07" ixz="1.2e-06" iyy="0.00141763" iyz="7.596e-05" izz="0.0001972"/>
     </inertial>
@@ -499,5 +416,5 @@
     <inertial>
       <mass value="0.457418" />
-      <origin xyz="-1.788e-05 0.00395812 -0.20273" rpy="0 -0 0"/>
+      <origin xyz="0.1 0.00395812 -0.00273" rpy="0 -0 0"/>
       <inertia ixx="0.00069205" ixy="-3e-08" ixz="5.2e-07" iyy="0.00068903" iyz="1.915e-05" izz="0.00013509"/>
     </inertial>
@@ -557,5 +474,5 @@
     <inertial>
       <mass value="1.05156" />
-      <origin xyz="-0.048476 3.2e-06 -0.0388988" rpy="0 -0 0"/>
+      <origin xyz="0.0 0.0 -0.08" rpy="0 -0 0"/>
       <inertia ixx="0.00194072" ixy="-1.1e-07" ixz="-0.00042482" iyy="0.00209392" iyz="-1.2e-07" izz="0.00035788"/>
     </inertial>
@@ -593,5 +510,5 @@
     <axis xyz="0 0 1"/>
     <limit lower="-1.5707963" upper="1.5707963" effort="150" velocity="1.0"/>
-    <dynamics damping="1.5" friction="0"/>
+    <dynamics damping="0.5" friction="0.5"/>
   </joint>
   <xacro:transmission_nx_joint name="LARM_JOINT1" />
@@ -602,5 +519,5 @@
     <axis xyz="0 1 0"/>
     <limit lower="-2.44346" upper="1.0471975" effort="150" velocity="1.0"/>
-    <dynamics damping="1.5" friction="0"/>
+    <dynamics damping="0.5" friction="0.5"/>
   </joint>
   <xacro:transmission_nx_joint name="LARM_JOINT2" />
@@ -611,5 +528,5 @@
     <axis xyz="0 1 0"/>
     <limit lower="-1.22173" upper="1.5707963" effort="150" velocity="1.0"/>
-    <dynamics damping="1.5" friction="0"/>
+    <dynamics damping="0.5" friction="0.5"/>
   </joint>
   <xacro:transmission_nx_joint name="LARM_JOINT3" />
@@ -620,5 +537,5 @@
     <axis xyz="1 0 0"/>
     <limit lower="-3.1415926" upper="1.7453292" effort="150" velocity="1.0"/>
-    <dynamics damping="1.5" friction="0"/>
+    <dynamics damping="0.5" friction="0.5"/>
   </joint>
   <xacro:transmission_nx_joint name="LARM_JOINT4" />
@@ -629,5 +546,5 @@
     <axis xyz="0 1 0"/>
     <limit lower="-3.57792" upper="1.134464" effort="150" velocity="1.0"/>
-    <dynamics damping="1.5" friction="0"/>
+    <dynamics damping="0.5" friction="0.5"/>
   </joint>
   <xacro:transmission_nx_joint name="LARM_JOINT5" />
@@ -637,6 +554,6 @@
     <origin xyz="0 0 -0.1335" rpy="0 0 0"/>
     <axis xyz="0 0 1"/>
-    <limit lower="-4.7123889" upper="4.7123889" effort="150" velocity="1.0"/>
-    <dynamics damping="1.5" friction="0"/>
+    <limit lower="-2.7123889" upper="2.7123889" effort="150" velocity="1.0"/>
+    <dynamics damping="0.5" friction="0.5"/>
   </joint>
   <xacro:transmission_nx_joint name="RARM_JOINT0" />
@@ -647,5 +564,5 @@
     <axis xyz="0 0 1"/>
     <limit lower="-1.570796" upper="1.570796" effort="150" velocity="1.0"/>
-    <dynamics damping="1.5" friction="0"/>
+    <dynamics damping="0.5" friction="0.5"/>
   </joint>
   <xacro:transmission_nx_joint name="RARM_JOINT1" />
@@ -656,5 +573,5 @@
     <axis xyz="0 1 0"/>
     <limit lower="-2.44346" upper="1.047197" effort="150" velocity="1.0"/>
-    <dynamics damping="1.5" friction="0"/>
+    <dynamics damping="0.5" friction="0.5"/>
   </joint>
   <xacro:transmission_nx_joint name="RARM_JOINT2" />
@@ -665,5 +582,5 @@
     <axis xyz="0 1 0"/>
     <limit lower="-1.22173" upper="1.570796" effort="150" velocity="1.0"/>
-    <dynamics damping="1.5" friction="0"/>
+    <dynamics damping="0.5" friction="0.5"/>
   </joint>
   <xacro:transmission_nx_joint name="RARM_JOINT3" />
@@ -674,5 +591,5 @@
     <axis xyz="1 0 0"/>
     <limit lower="-1.74532" upper="3.141592" effort="150" velocity="1.0"/>
-    <dynamics damping="1.5" friction="0"/>
+    <dynamics damping="0.5" friction="0.5"/>
   </joint>
   <xacro:transmission_nx_joint name="RARM_JOINT4" />
@@ -683,5 +600,5 @@
     <axis xyz="0 1 0"/>
     <limit lower="-3.5779" upper="1.134464" effort="150" velocity="1.0"/>
-    <dynamics damping="1.5" friction="0"/>
+    <dynamics damping="0.5" friction="0.5"/>
   </joint>
   <xacro:transmission_nx_joint name="RARM_JOINT5" />
@@ -691,14 +608,56 @@
     <origin xyz="0 0 -0.1335" rpy="0 0 0"/>
     <axis xyz="0 0 1"/>
-    <limit lower="-4.712388" upper="4.712388" effort="150" velocity="1.0"/>
-    <dynamics damping="1.5" friction="0"/>
+    <limit lower="-2.712388" upper="2.712388" effort="150" velocity="1.0"/>
+    <dynamics damping="0.5" friction="0.5"/>
   </joint>
   <!-- Gazebo plugin for ROS Control -->
   <gazebo>
-    <plugin name="gazebo_ros_control" filename="libgazebo_ros_control.so">
-      <robotNamespace>/</robotNamespace>
-      <robotSimType>gazebo_ros_control/DefaultRobotHWSim</robotSimType>
-    </plugin>
-    <dampingFactor>0.8</dampingFactor>
+    <plugin name="gazebo_ros_control" filename="libgazebo_ros_control.so" />
+  </gazebo>
+  <!-- Gazebo-Specific Link Properties -->
+  <gazebo reference="CHEST_JOINT0">
+    <implicitSpringDamper>1</implicitSpringDamper>
+  </gazebo>
+  <gazebo reference="HEAD_JOINT0">
+    <implicitSpringDamper>1</implicitSpringDamper>
+  </gazebo>
+  <gazebo reference="HEAD_JOINT1">
+    <implicitSpringDamper>1</implicitSpringDamper>
+  </gazebo>
+  <gazebo reference="LARM_JOINT0">
+    <implicitSpringDamper>1</implicitSpringDamper>
+  </gazebo>
+  <gazebo reference="LARM_JOINT1">
+    <implicitSpringDamper>1</implicitSpringDamper>
+  </gazebo>
+  <gazebo reference="LARM_JOINT2">
+    <implicitSpringDamper>1</implicitSpringDamper>
+  </gazebo>
+  <gazebo reference="LARM_JOINT3">
+    <implicitSpringDamper>1</implicitSpringDamper>
+  </gazebo>
+  <gazebo reference="LARM_JOINT4">
+    <implicitSpringDamper>1</implicitSpringDamper>
+  </gazebo>
+  <gazebo reference="LARM_JOINT5">
+    <implicitSpringDamper>1</implicitSpringDamper>
+  </gazebo>
+  <gazebo reference="RARM_JOINT0">
+    <implicitSpringDamper>1</implicitSpringDamper>
+  </gazebo>
+  <gazebo reference="RARM_JOINT1">
+    <implicitSpringDamper>1</implicitSpringDamper>
+  </gazebo>
+  <gazebo reference="RARM_JOINT2">
+    <implicitSpringDamper>1</implicitSpringDamper>
+  </gazebo>
+  <gazebo reference="RARM_JOINT3">
+    <implicitSpringDamper>1</implicitSpringDamper>
+  </gazebo>
+  <gazebo reference="RARM_JOINT4">
+    <implicitSpringDamper>1</implicitSpringDamper>
+  </gazebo>
+  <gazebo reference="RARM_JOINT5">
+    <implicitSpringDamper>1</implicitSpringDamper>
   </gazebo>
 </robot>

Commit message: split hand-camera links

File: nextagea_description/urdf/NextageA_robot.xacro (robot description, xacro)
@@ -276,20 +276,8 @@
       </geometry>
     </visual>
-    <visual>
-      <origin xyz="0 0 0" rpy="0 0 0"/>
-      <geometry>
-	      <mesh filename="package://nextagea_description/urdf/meshes/L_CAM.dae"/>
-      </geometry>
-    </visual>
-    <collision>
-      <origin xyz="0 0 -0.02" rpy="0 0 0"/>
-      <geometry>
-        <cylinder length="0.07" radius="0.037"/>
-      </geometry>
-    </collision>
-    <collision>
-      <origin xyz="0.0525 0.029 -0.02" rpy="0 0 0"/>
-      <geometry>
-        <box size="0.057 0.106 0.042"/>
+    <collision>
+      <origin xyz="0 0 0.0065" rpy="0 0 0"/>
+      <geometry>
+        <cylinder length="0.013" radius="0.037"/>
       </geometry>
     </collision>
@@ -300,4 +288,30 @@
     </inertial>
   </link>
+  <xacro:gazebo_nx_link name="LARM_camera_Link" color="Black" />
+  <link name="LARM_camera_Link">
+    <visual>
+      <origin xyz="0 0 0" rpy="0 0 0"/>
+      <geometry>
+        <mesh filename="package://nextagea_description/urdf/meshes/L_CAM.dae"/>
+      </geometry>
+    </visual>
+    <collision>
+      <origin xyz="0 0 -0.025" rpy="0 0 0"/>
+      <geometry>
+        <cylinder length="0.05" radius="0.037"/>
+      </geometry>
+    </collision>
+    <collision>
+      <origin xyz="0.0525 0.029 -0.02" rpy="0 0 0"/>
+      <geometry>
+        <box size="0.057 0.106 0.042"/>
+      </geometry>
+    </collision>
+    <inertial>
+      <mass value="1.05156" />
+      <origin xyz="0.0 0.0 -0.08" rpy="0 -0 0"/>
+      <inertia ixx="0.00194072" ixy="1.1e-07" ixz="-0.00042482" iyy="0.00209392" iyz="1.2e-07" izz="0.00035788"/>
+    </inertial>
+  </link>
   <xacro:gazebo_nx_link name="RARM_JOINT0_Link" color="Black" />
   <link name="RARM_JOINT0_Link">
@@ -456,14 +470,28 @@
       </geometry>
     </visual>
-    <visual>
-      <origin xyz="0 0 0" rpy="0 0 0"/>
-      <geometry>
-	      <mesh filename="package://nextagea_description/urdf/meshes/R_CAM.dae"/>
-      </geometry>
-    </visual>
-    <collision>
-      <origin xyz="0 0 -0.02" rpy="0 0 0"/>
-      <geometry>
-        <cylinder length="0.07" radius="0.037"/>
+    <collision>
+      <origin xyz="0 0 0.0065" rpy="0 0 0"/>
+      <geometry>
+        <cylinder length="0.013" radius="0.037"/>
+      </geometry>
+    </collision>
+    <inertial>
+      <mass value="1.05156" />
+      <origin xyz="0.0 0.0 -0.08" rpy="0 -0 0"/>
+      <inertia ixx="0.00194072" ixy="-1.1e-07" ixz="-0.00042482" iyy="0.00209392" iyz="-1.2e-07" izz="0.00035788"/>
+    </inertial>
+  </link>
+  <xacro:gazebo_nx_link name="RARM_camera_Link" color="Black" />
+  <link name="RARM_camera_Link">
+    <visual>
+      <origin xyz="0 0 0" rpy="0 0 0"/>
+      <geometry>
+        <mesh filename="package://nextagea_description/urdf/meshes/R_CAM.dae"/>
+      </geometry>
+    </visual>
+    <collision>
+      <origin xyz="0 0 -0.025" rpy="0 0 0"/>
+      <geometry>
+        <cylinder length="0.05" radius="0.037"/>
       </geometry>
     </collision>
@@ -559,4 +587,10 @@
     <dynamics damping="0.5" friction="0.5"/>
   </joint>
+  <joint name="LARM_JOINT6" type="fixed">
+    <parent link="LARM_JOINT5_Link"/>
+    <child link="LARM_camera_Link"/>
+    <origin xyz="0 0 0" rpy="0 0 0"/>
+    <axis xyz="0 0 1"/>
+  </joint>
   <xacro:transmission_nx_joint name="RARM_JOINT0" />
   <joint name="RARM_JOINT0" type="revolute">
@@ -612,4 +646,10 @@
     <limit lower="-2.712388" upper="2.712388" effort="150" velocity="1.0"/>
     <dynamics damping="0.5" friction="0.5"/>
+  </joint>
+  <joint name="RARM_JOINT6" type="fixed">
+    <parent link="RARM_JOINT5_Link"/>
+    <child link="RARM_camera_Link"/>
+    <origin xyz="0 0 0" rpy="0 0 0"/>
+    <axis xyz="0 0 1"/>
   </joint>
   <!-- Gazebo plugin for ROS Control -->
