Commit message: split camera links out of main robot xacro

File: nextagea_description/urdf/NextageAOpen.urdf.xacro (robot description, xacro)
@@ -18,3 +18,45 @@
   <xacro:include filename="$(find nextagea_description)/urdf/NextageA_base.xacro" />
   <xacro:include filename="$(find nextagea_description)/urdf/NextageA_robot.xacro" />
+  <xacro:macro name="nxao_camera" params="prefix parent">
+    <xacro:if value="${prefix == 'L'}">
+      <xacro:property name="m" value="+1" />
+    </xacro:if>
+    <xacro:if value="${prefix == 'R'}">
+      <xacro:property name="m" value="-1" />
+    </xacro:if>
+    <xacro:gazebo_nx_link name="${prefix}ARM_camera_Link" color="Black" />
+    <link name="${prefix}ARM_camera_Link">
+      <visual>
+        <origin xyz="0 0 0" rpy="0 0 0"/>
+        <geometry>
+          <mesh filename="package://nextagea_description/urdf/meshes/${prefix}_CAM.dae"/>
+        </geometry>
+      </visual>
+      <collision>
+        <origin xyz="0 0 -0.025" rpy="0 0 0"/>
+        <geometry>
+          <cylinder length="0.05" radius="0.037"/>
+        </geometry>
+      </collision>
+      <collision>
+        <origin xyz="0.0525 ${m * 0.029} -0.02" rpy="0 0 0"/>
+        <geometry>
+          <box size="0.057 0.106 0.042"/>
+        </geometry>
+      </collision>
+      <inertial>
+        <mass value="1.05156" />
+        <origin xyz="0.0 0.0 -0.08" rpy="0 -0 0"/>
+        <inertia ixx="0.00194072" ixy="${m * 1.1e-07}" ixz="-0.00042482" iyy="0.00209392" iyz="${m * 1.2e-07}" izz="0.00035788"/>
+      </inertial>
+    </link>
+    <joint name="${prefix}ARM_JOINT6" type="fixed">
+      <parent link="${parent}"/>
+      <child link="${prefix}ARM_camera_Link"/>
+      <origin xyz="0 0 0" rpy="0 0 0"/>
+      <axis xyz="0 0 1"/>
+    </joint>
+  </xacro:macro>
+  <xacro:nxao_camera prefix="L" parent="LARM_JOINT5_Link" />
+  <xacro:nxao_camera prefix="R" parent="RARM_JOINT5_Link" />
 </robot>

File: nextagea_description/urdf/NextageA_robot.xacro (robot description, xacro)
@@ -288,30 +288,4 @@
     </inertial>
   </link>
-  <xacro:gazebo_nx_link name="LARM_camera_Link" color="Black" />
-  <link name="LARM_camera_Link">
-    <visual>
-      <origin xyz="0 0 0" rpy="0 0 0"/>
-      <geometry>
-        <mesh filename="package://nextagea_description/urdf/meshes/L_CAM.dae"/>
-      </geometry>
-    </visual>
-    <collision>
-      <origin xyz="0 0 -0.025" rpy="0 0 0"/>
-      <geometry>
-        <cylinder length="0.05" radius="0.037"/>
-      </geometry>
-    </collision>
-    <collision>
-      <origin xyz="0.0525 0.029 -0.02" rpy="0 0 0"/>
-      <geometry>
-        <box size="0.057 0.106 0.042"/>
-      </geometry>
-    </collision>
-    <inertial>
-      <mass value="1.05156" />
-      <origin xyz="0.0 0.0 -0.08" rpy="0 -0 0"/>
-      <inertia ixx="0.00194072" ixy="1.1e-07" ixz="-0.00042482" iyy="0.00209392" iyz="1.2e-07" izz="0.00035788"/>
-    </inertial>
-  </link>
   <xacro:gazebo_nx_link name="RARM_JOINT0_Link" color="Black" />
   <link name="RARM_JOINT0_Link">
@@ -474,30 +448,4 @@
       <geometry>
         <cylinder length="0.013" radius="0.037"/>
-      </geometry>
-    </collision>
-    <inertial>
-      <mass value="1.05156" />
-      <origin xyz="0.0 0.0 -0.08" rpy="0 -0 0"/>
-      <inertia ixx="0.00194072" ixy="-1.1e-07" ixz="-0.00042482" iyy="0.00209392" iyz="-1.2e-07" izz="0.00035788"/>
-    </inertial>
-  </link>
-  <xacro:gazebo_nx_link name="RARM_camera_Link" color="Black" />
-  <link name="RARM_camera_Link">
-    <visual>
-      <origin xyz="0 0 0" rpy="0 0 0"/>
-      <geometry>
-        <mesh filename="package://nextagea_description/urdf/meshes/R_CAM.dae"/>
-      </geometry>
-    </visual>
-    <collision>
-      <origin xyz="0 0 -0.025" rpy="0 0 0"/>
-      <geometry>
-        <cylinder length="0.05" radius="0.037"/>
-      </geometry>
-    </collision>
-    <collision>
-      <origin xyz="0.0525 -0.029 -0.02" rpy="0 0 0"/>
-      <geometry>
-        <box size="0.057 0.106 0.042"/>
       </geometry>
     </collision>
@@ -587,10 +535,4 @@
     <dynamics damping="0.5" friction="0.5"/>
   </joint>
-  <joint name="LARM_JOINT6" type="fixed">
-    <parent link="LARM_JOINT5_Link"/>
-    <child link="LARM_camera_Link"/>
-    <origin xyz="0 0 0" rpy="0 0 0"/>
-    <axis xyz="0 0 1"/>
-  </joint>
   <xacro:transmission_nx_joint name="RARM_JOINT0" />
   <joint name="RARM_JOINT0" type="revolute">
@@ -646,10 +588,4 @@
     <limit lower="-2.712388" upper="2.712388" effort="150" velocity="1.0"/>
     <dynamics damping="0.5" friction="0.5"/>
-  </joint>
-  <joint name="RARM_JOINT6" type="fixed">
-    <parent link="RARM_JOINT5_Link"/>
-    <child link="RARM_camera_Link"/>
-    <origin xyz="0 0 0" rpy="0 0 0"/>
-    <axis xyz="0 0 1"/>
   </joint>
   <!-- Gazebo plugin for ROS Control -->

Commit message: define and activate FT-sensor link

File: nextagea_description/urdf/NextageAOpen.urdf.xacro (robot description, xacro)
@@ -18,4 +18,6 @@
   <xacro:include filename="$(find nextagea_description)/urdf/NextageA_base.xacro" />
   <xacro:include filename="$(find nextagea_description)/urdf/NextageA_robot.xacro" />
+  <xacro:arg name="use_hand_cameras" default="false"/>
+  <xacro:arg name="use_ft_sensors" default="false"/>
   <xacro:macro name="nxao_camera" params="prefix parent">
     <xacro:if value="${prefix == 'L'}">
@@ -58,5 +60,52 @@
     </joint>
   </xacro:macro>
-  <xacro:nxao_camera prefix="L" parent="LARM_JOINT5_Link" />
-  <xacro:nxao_camera prefix="R" parent="RARM_JOINT5_Link" />
+  <xacro:macro name="nxao_ft_sensor" params="prefix parent">
+    <xacro:if value="${prefix == 'L'}">
+      <xacro:property name="m" value="+1" />
+    </xacro:if>
+    <xacro:if value="${prefix == 'R'}">
+      <xacro:property name="m" value="-1" />
+    </xacro:if>
+    <xacro:gazebo_nx_link name="${prefix}ARM_ft_Link" color="LightGrey" />
+    <link name="${prefix}ARM_ft_Link">
+      <visual>
+        <origin xyz="0 0 0.0185" rpy="0 0 0"/>
+        <geometry>
+          <cylinder length="0.037" radius="0.035"/>
+        </geometry>
+        <material name="LightGrey">
+          <color rgba="0.6 0.6 0.6 1.0"/>
+        </material>
+      </visual>
+      <collision>
+        <origin xyz="0 0 0.0185" rpy="0 0 0"/>
+        <geometry>
+          <cylinder length="0.037" radius="0.04"/>
+        </geometry>
+      </collision>
+      <!-- TODO: The inertial values are copied from ARM_JOINT5_Link. Replace with proper values. -->
+      <inertial>
+        <mass value="1.05156" />
+        <origin xyz="0.0 0.0 -0.08" rpy="0 -0 0"/>
+        <inertia ixx="0.00194072" ixy="1.1e-07" ixz="-0.00042482" iyy="0.00209392" iyz="1.2e-07" izz="0.00035788"/>
+      </inertial>
+    </link>
+    <joint name="${prefix}ARM_ft_joint" type="fixed">
+      <parent link="${parent}"/>
+      <child link="${prefix}ARM_ft_Link"/>
+      <origin xyz="0 0 -0.037" rpy="0 0 0"/>
+      <axis xyz="0 0 1"/>
+    </joint>
+  </xacro:macro>
+  <xacro:property name="arm_tip" value="ARM_JOINT5_Link" />
+  <xacro:if value="$(arg use_ft_sensors)">
+    <xacro:nxao_ft_sensor prefix="L" parent="L${arm_tip}" />
+    <xacro:nxao_ft_sensor prefix="R" parent="R${arm_tip}" />
+    <xacro:property name="arm_tip" value="ARM_ft_Link" />
+  </xacro:if>
+  <xacro:if value="$(arg use_hand_cameras)">
+    <xacro:nxao_camera prefix="L" parent="L${arm_tip}" />
+    <xacro:nxao_camera prefix="R" parent="R${arm_tip}" />
+    <xacro:property name="arm_tip" value="ARM_camera_Link" />
+  </xacro:if>
 </robot>

File: nextagea_description/urdf/NextageAOpen_gazebo_intel_realsense.urdf.xacro (robot description, xacro)
@@ -3,4 +3,6 @@
        xmlns:xacro="http://www.ros.org/wiki/xacro">
   <xacro:property name="fixed_base" value="True" />
+  <xacro:property name="ft_sensors" value="True" />
+  <xacro:property name="hand_camera" value="True" />
   <xacro:include filename="$(find nextagea_description)/urdf/NextageAOpen_gazebo.urdf.xacro" />
   <xacro:include filename="$(find realsense2_description)/urdf/_d435.urdf.xacro"/>
